File: kicad/ESL-scourge.sch (KiCad schematic (older format))
At the start: 45 parts, among them IC1 MOC3020M, J1 DB9, J2 DB9, P1 CONN_4, P2 CONN_3, P3 CONN_4, Q1 BC847, Q2 BC847, Q3 BC847, U1 TDA2030

Commit message: Add initial maket_lovat as a separate branch (kicad folder only)
Parts:
- removed C? (x2): 22x350 12-18mm, ~, symbol CP1
- removed D10, D6, D7, D8, D9, D?: SMA4007 (GS1M), ~, symbol DIODE
- removed D5: LED, ~, symbol LED
- removed IC1: MOC3020M, DIP6, symbol MOC3020M
- removed J1, J2: DB9, symbol DB9
- removed JP1: JUMPER, ~, symbol JUMPER
- removed P1, P3: CONN_4, symbol CONN_4
- removed P2: CONN_3, symbol CONN_3
- removed Q1, Q2, Q3: BC847, ~, symbol NPN
- removed R10: 0*, ~, symbol R
- removed R11: 10k, ~, symbol R
- removed R12, R13: 30k, ~, symbol R
- removed R8: 1M*, ~, symbol R
- removed R9: 2k*, ~, symbol R
- removed RV?: SH-855MC, 100k, ~, symbol POT
- added P1, P2: CONN_2, symbol CONN_2
- added T1: ТПК-1 (2х9В, 0.08А) (ТПГ-1), ~, symbol TRANSFO2
- added T2: ТПК-1 (18В, 0.08А) (ТПГ-1), ~, symbol TRANSFO
- C1: value 1000.0x35V 13mm -> 1000.0x25V
- C3: renamed from C6; value 1.0 x 250V -> 1.0
- C5: renamed from C4; value 2200.0x35V 16-18mm -> 2200.0x25V
- D1, D2, D3, D4: value SMA4007 (GS1M) -> DIODE
- R5: renamed from R6; value ? -> 100k
- R6: renamed from R7; value 10k -> 100k
- renumbered C3 to C4, C5 to C6, R5 to R7
Connections:
- net GND: now also C3.2, T1.4 (SB), T1.5 (SC), T2.4 (SB)
- net at C5.1, D3.1 (A), D4.2 (K)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: now also R6.2; no longer U1.2 (IN-)
- net at C5.2, R7.1: now also T2.3 (SA)
- net at R6.1: now also R5.1, U1.2 (IN-)
- net at R5.2: now also C3.1
- net at D1.1 (A), R1.1: now also T1.3 (SA)
- net at D2.1 (A): now also C1.1, C4.1, D1.2 (K), D3.2 (K), R3.1, U1.5 (VCC)
- removed net VCC: C1.1, C4.1, D1.2 (K), D2.2 (K), D3.2 (K), R3.1, R5.1, U1.5 (VCC)
- new net: P1.2 (PM), T1.1 (AA)
- new net: P1.1 (P1), T1.2 (AB)
- new net: D2.2 (K), T1.6 (SD)
- new net: P2.2 (PM), T2.1 (AA)
- new net: P2.1 (P1), T2.2 (AB)
Other:
- note removed: "*"
- note removed: "12V"
- note removed: "15ма"
- note removed: "220V"
- note removed: "R1 и R2 подбираются так, чтобы\nАМПЛИТУДНОЕ выходное\nнапряжение менялось в диапазоне\nне менее, чем 20-100 В.\nС помощью осциллографа с\nделителем убедиться, что\nсинус на выходе не срезается."
- note removed: "R6=(Vcc-4)/0,015, округляется в\nсторону уменьшения до близжайшего\nдоступного номинала, но не менее,\nчем (Vcc-2)/0,05\n"
- note removed: "Если вольтметр на 150В:\nR10 - 0 ом (перемычка)\nR8 - 1M или не монтировать вообще\n(посмотреть, насколько бодро\nвольтметр реагирует на вращение\nрегулятора напряжения)."
- note removed: "Заменить на db15, сделать совместимым с тредбаном"
- note removed: "Здесь важна фазировка обмоток:\nнапряжения должны суммироваться,\nа не вычитаться. Необходимо\nизмерить переменное напряжение\nмежду выводами 1 и 4 P1\n - если там 24 В - все ОК\n - если там около нуля, необходимо\nпоменять местами концы одной из\nвторичных обмоток.\nПредварительно надо убедиться,\nчто на каждой из обмоток есть 12 В."
- note removed: "По умолчанию установлен (замкнут)"
- note removed: "Посмотреть выходной сигнал\nс отключенным демпфером (R5C5).\nЕсли все ОК - демпфер не ставить."
- note removed: "ТТП-30 (2х18В, 0.75А)\n(лучше ТТП-15 2х18В, но его не найти)"
- note removed: "Торэл ТТП-3 (12В, 0.2А)"
- note removed: "для подбора R9 сделать следующее:\nпри максимальном напряжении на\nвыходе замкнуть контакты 7 и 8\nили лучше замкнуть контакт 8 с\nножкой 6 IC1. Если напряжение на\nвольтметре карабаса уменьшилось\nнезначительно - ОК."
- note removed: "может быть заменить на КМОП-логику?"
- note removed: "может быть стоит подключить\nвольтметр до резистора тк мб кз\nили предусмотреть индикацию КЗ?"
- note removed: "переделать на инвертирующий?"
- note removed: "предусмотреть, но не ставить"
- moved on the sheet: C3, R5, R6
